Commit message: last version

File: my_robot_description/urdf/mobile_base.xacro (robot description, xacro)
@@ -3,5 +3,5 @@
     <xacro:property name="base_length" value="0.6" />
     <xacro:property name="base_width" value="0.4" />
-    <xacro:property name="base_height" value="0.2" />
+    <xacro:property name="base_height" value="0.2" /><!--meters-->
     <xacro:property name="base_mass" value="5.0" /> <!--Kg-->
     <xacro:property name="wheel_mass" value="1.0" />
